Commit message: Can drive sim rover now, but buggy cmd_vel translator

File: rover_description/rover_desc/rover.urdf (robot description, URDF)
Before this commit: robot rover, 23 links, 22 joints
Links:
- link bl_clamp: geometry collision mesh filename=package://rover_description/rover_desc/parts/bl_clamp.stl; visual mesh filename=package://rover_description/rover_desc/parts/bl_clamp.stl
- link bl_motor: geometry collision mesh filename=package://rover_description/rover_desc/parts/bl_motor.stl; visual mesh filename=package://rover_description/rover_desc/parts/bl_motor.stl
- link bl_servo: geometry collision mesh filename=package://rover_description/rover_desc/parts/bl_servo.stl; visual mesh filename=package://rover_description/rover_desc/parts/bl_servo.stl
- link bl_steer: geometry collision mesh filename=package://rover_description/rover_desc/parts/bl_steer.stl; visual mesh filename=package://rover_description/rover_desc/parts/bl_steer.stl
- link bl_whl: geometry collision mesh filename=package://rover_description/rover_desc/parts/bl_whl.stl; visual mesh filename=package://rover_description/rover_desc/parts/bl_whl.stl
- link body: geometry collision mesh filename=package://rover_description/rover_desc/parts/body.stl; visual mesh filename=package://rover_description/rover_desc/parts/body.stl
- link br_clamp: geometry collision mesh filename=package://rover_description/rover_desc/parts/br_clamp.stl; visual mesh filename=package://rover_description/rover_desc/parts/br_clamp.stl
- link br_motor: geometry collision mesh filename=package://rover_description/rover_desc/parts/br_motor.stl; visual mesh filename=package://rover_description/rover_desc/parts/br_motor.stl
- link br_servo: geometry collision mesh filename=package://rover_description/rover_desc/parts/br_servo.stl; visual mesh filename=package://rover_description/rover_desc/parts/br_servo.stl
- link br_steer: geometry collision mesh filename=package://rover_description/rover_desc/parts/br_steer.stl; visual mesh filename=package://rover_description/rover_desc/parts/br_steer.stl
- link br_whl: geometry collision mesh filename=package://rover_description/rover_desc/parts/br_whl.stl; visual mesh filename=package://rover_description/rover_desc/parts/br_whl.stl
- link fl_clamp: geometry collision mesh filename=package://rover_description/rover_desc/parts/fl_clamp.stl; visual mesh filename=package://rover_description/rover_desc/parts/fl_clamp.stl
- link fl_motor: geometry collision mesh filename=package://rover_description/rover_desc/parts/fl_motor.stl; visual mesh filename=package://rover_description/rover_desc/parts/fl_motor.stl
- link fl_servo: geometry collision mesh filename=package://rover_description/rover_desc/parts/fl_servo.stl; visual mesh filename=package://rover_description/rover_desc/parts/fl_servo.stl
- link fl_steer: geometry collision mesh filename=package://rover_description/rover_desc/parts/fl_steer.stl; visual mesh filename=package://rover_description/rover_desc/parts/fl_steer.stl
- link fl_whl: geometry collision mesh filename=package://rover_description/rover_desc/parts/fl_whl.stl; visual mesh filename=package://rover_description/rover_desc/parts/fl_whl.stl
- link fr_clamp: geometry collision mesh filename=package://rover_description/rover_desc/parts/fr_clamp.stl; visual mesh filename=package://rover_description/rover_desc/parts/fr_clamp.stl
- link fr_motor: geometry collision mesh filename=package://rover_description/rover_desc/parts/fr_motor.stl; visual mesh filename=package://rover_description/rover_desc/parts/fr_motor.stl
- link fr_servo: geometry collision mesh filename=package://rover_description/rover_desc/parts/fr_servo.stl; visual mesh filename=package://rover_description/rover_desc/parts/fr_servo.stl
- link fr_steer: geometry collision mesh filename=package://rover_description/rover_desc/parts/fr_steer.stl; visual mesh filename=package://rover_description/rover_desc/parts/fr_steer.stl
- link fr_whl: geometry collision mesh filename=package://rover_description/rover_desc/parts/fr_whl.stl; visual mesh filename=package://rover_description/rover_desc/parts/fr_whl.stl
- link left_rocker: geometry collision mesh filename=package://rover_description/rover_desc/parts/left_rocker.stl; visual mesh filename=package://rover_description/rover_desc/parts/left_rocker.stl
- link right_rocker: geometry collision mesh filename=package://rover_description/rover_desc/parts/right_rocker.s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; visual mesh filename=package://rover_description/rover_desc/parts/right_rocker.s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
