Commit message: Finally got the mfin realsense simulated holy fuck

File: rover_description/rover_desc/gazebo_params.xacro (robot description, xacro)
@@ -52,21 +52,49 @@
     <gazebo reference="fr_whl">
         <material>Gazebo/Black</material>
-        <mu1 value="10"/>
-        <mu2 value="10"/>
+        <mu1 value="1"/>
+        <mu2 value="1"/>
     </gazebo>
     <gazebo reference="fl_whl">
         <material>Gazebo/Black</material>
-        <mu1 value="10"/>
-        <mu2 value="10"/>
+        <mu1 value="1"/>
+        <mu2 value="1"/>
     </gazebo>
     <gazebo reference="br_whl">
         <material>Gazebo/Black</material>
-        <mu1 value="10"/>
-        <mu2 value="10"/>
+        <mu1 value="1"/>
+        <mu2 value="1"/>
     </gazebo>
     <gazebo reference="bl_whl">
         <material>Gazebo/Black</material>
-        <mu1 value="10"/>
-        <mu2 value="10"/>
+        <mu1 value="1"/>
+        <mu2 value="1"/>
+    </gazebo>
+    <gazebo reference="l_rocker2body">
+        <provideFeedback>true</provideFeedback>
+        <implicitSpringDamper>true</implicitSpringDamper>
+        <springStiffness>700.0</springStiffness>
+        <springReference>0.0</springReference>
+    </gazebo>
+    <gazebo reference="r_rocker2body">
+        <provideFeedback>true</provideFeedback>
+        <implicitSpringDamper>true</implicitSpringDamper>
+        <springStiffness>700.0</springStiffness>
+        <springReference>0.0</springReference>
+        <friction>0.75</friction>
+    </gazebo>
+    <!-- These are temporary just to stop them from flopping around -->
+    <gazebo reference="rs_yaw">
+        <provideFeedback>true</provideFeedback>
+        <implicitSpringDamper>true</implicitSpringDamper>
+        <springStiffness>700.0</springStiffness>
+        <springReference>0.0</springReference>
+        <friction>0.75</friction>
+    </gazebo>
+    <gazebo reference="rs_pitch">
+        <provideFeedback>true</provideFeedback>
+        <implicitSpringDamper>true</implicitSpringDamper>
+        <springStiffness>700.0</springStiffness>
+        <springReference>0.0</springReference>
+        <friction>0.75</friction>
     </gazebo>
 </robot>

File: rover_description/rover_desc/rover.xacro (robot description, xacro)
@@ -2,7 +2,17 @@
 <robot xmlns:xacro="http://ros.org/wiki/xacro" name="rover">
     <!-- URDF & Visual -->
-    <xacro:include filename="$(find rover_description)/rover_desc/rover.urdf" />
-    <xacro:include filename="$(find rover_description)/rover_desc/gazebo_colors.xacro" />
+    <xacro:include filename="$(find rover_description)/rover_desc/parts/robot.urdf" />
+    <xacro:include filename="$(find rover_description)/rover_desc/gazebo_params.xacro" />
+    <xacro:include filename="$(find rover_description)/rover_desc/realsense.urdf" />
+    <xacro:include filename="$(find rover_description)/rover_desc/gz_realsense.xacro"/>
+    <xacro:realsense_d435 parent="imager_3">
+        <origin xyz="-0.0325 0 -0.005" rpy="${pi/2} ${pi/2} ${0}"/>
+    </xacro:realsense_d435>
+    <!-- <joint name="rs_to_rover" type="fixed">
+        <parent link="rover_base" />
+        <child link="base_link" />
+    </joint> -->
     <!-- Include ros2_control -->
-    <xacro:include filename="$(find rover_gz)/plugins/ros2_control.xacro" />
+    <!-- <xacro:include filename="$(find rover_gz)/plugins/ros2_control.xacro" /> -->
+    <!-- <xacro:include filename="$(find rover_description)/rover_desc/parts/imu.xacro" /> -->
 </robot>
